File: laser-driver-ic-nzn.kicad_pcb (KiCad board)
At the start: 2 copper layers, 76 x 75.5 mm, 18 parts, among them J1 Laser connector (PD-30S), J2 12V input, J3 RF I, J4 RF Q, J5 REF, U1 IC-NZN QFN24-4X4, U2 AD5274BRM, U3 AD5274BRM, U4 LM78M05_TO252

Commit message: Finalize v0.1 for manufacture
Routing:
- net Net-(U2-W): track 7.92 -> 14.7 mm
- net GND: track 89.6 -> 84.5 mm
- net /Chip wakeup: track 48.9 -> 48.2 mm
